File: kicad/esp32board.sch (KiCad schematic (older format))
At the start: 33 parts, among them P1 ADC, P2 ADC_TOUCH, U0 SERIAL1, U1 SERIAL2

Commit message: Added I2S amplifier (Incomplete)
Parts:
- removed JP1: Jumper_NC_Dual, symbol Jumper_NC_Dual
- removed U0: SERIAL1, Pin_Headers:Pin_Header_Straight_1x04, symbol CONN_01X04
- added C10: .1uF, Capacitors_SMD:C_0603_HandSoldering, symbol C
- added I2S: MAX98357A, MODULE, symbol MAX98357A
- added JP_MPU_FSYNC1: JP_NO, jumper:SOLDER-JUMPER_1-WAY, symbol Jumper_NO_Small
- added R3, R4: 100K, Resistors_SMD:R_0603_HandSoldering, symbol R
- added SPK: CONN_SPK, symbol CONN_01X02
- JP_MPU_INT1: footprint jumper:SOLDER-JUMPER_2-WAY -> jumper:SOLDER-JUMPER_1-WAY
Connections:
- net +3V3: now also C10.1
- net +5V: now also I2S.4 (SD_MODE), I2S.7 (Vdd), I2S.8 (Vdd)
- net ADC_0: now also I2S.1 (DIN)
- net ADC_1: now also I2S.14 (LRCLK), JP_MPU_FSYNC1.2
- net ADC_2: now also I2S.16 (BCLK)
- net GND: now also C10.2, I2S.11 (GND), I2S.15 (GND), I2S.3 (GND), R3.1, R4.2
- net at MPU1.11 (FSYNC): now also JP_MPU_FSYNC1.1, R3.2
- new net: I2S.10 (OUTN), SPK.1 (P1)
- new net: I2S.2 (GAIN_SLOT), R4.1
- new net: I2S.9 (OUTP), SPK.2 (P2)
Changed lines of the file:
@@
 LIBS:ESP32-footprints-Shem-Lib
 LIBS:tinkerforge
+LIBS:MAX98357A
 LIBS:INA220
 LIBS:esp32board-cache
@@
 Text GLabel 6600 4450 2    60   Input ~ 0
 GND
-Text GLabel 4750 4500 0    60   Input ~ 0
+Text GLabel 4000 4500 0    60   Input ~ 0
 GND
 Text GLabel 5250 4850 3    60   Input ~ 0
 GND
-Text GLabel 4750 3200 0    60   Input ~ 0
+Text GLabel 4000 3200 0    60   Input ~ 0
 3.3V
 Text GLabel 2300 4950 2    60   Input ~ 0
@@
 U2_TX
 $Comp
-L CONN_01X04 U0
-U 1 1 595D3346
-P 3100 3850
-F 0 "U0" H 3100 4100 50  0000 C CNN
-F 1 "SERIAL1" V 3200 3850 50  0000 C CNN
-F 2 "Pin_Headers:Pin_Header_Straight_1x04" H 3100 3850 50  0001 C CNN
-F 3 "" H 3100 3850 50  0000 C CNN
-	1    3100 3850
-	-1   0    0    1
-$EndComp
-$Comp
 L CONN_01X04 U1
 U 1 1 595D349E
@@
 	-1   0    0    1
 $EndComp
-Text GLabel 3300 4000 2    60   Input ~ 0
-GND
-Text GLabel 3300 3800 2    60   Input ~ 0
-U0_RX
-Text GLabel 3300 3700 2    60   Input ~ 0
-U0_TX
-Text GLabel 3300 3900 2    60   Input ~ 0
-3.3V
 Text GLabel 6600 3050 2    60   Input ~ 0
 SPI_MOSI
@@
 F 0 "JP_MPU_INT1" H 10400 3280 50  0000 C CNN
 F 1 "JP_NO" H 10410 3140 50  0000 C CNN
-F 2 "jumper:SOLDER-JUMPER_2-WAY" H 10400 3200 50  0001 C CNN
+F 2 "jumper:SOLDER-JUMPER_1-WAY" H 10400 3200 50  0001 C CNN
 F 3 "" H 10400 3200 50  0000 C CNN
 	1    10400 3200
@@
 Wire Wire Line
 	10050 3050 10050 3700
-$Comp
-L Jumper_NC_Dual JP1
-U 1 1 59824C70
-P 10350 3700
-F 0 "JP1" H 10400 3600 50  0000 L CNN
-F 1 "Jumper_NC_Dual" H 10350 3800 50  0000 C BNN
-F 2 "" H 10350 3700 50  0000 C CNN
-F 3 "" H 10350 3700 50  0000 C CNN
-	1    10350 3700
+Wire Wire Line
+	10050 3700 10300 3700
+$Comp
+L R R3
+U 1 1 598A220A
+P 10600 3450
+F 0 "R3" V 10680 3450 50  0000 C CNN
+F 1 "100K" V 10600 3450 50  0000 C CNN
+F 2 "Resistors_SMD:R_0603_HandSoldering" V 10530 3450 50  0001 C CNN
+F 3 "" H 10600 3450 50  0000 C CNN
+	1    10600 3450
 	0    1    1    0
 $EndComp
 Wire Wire Line
-	10750 3450 10350 3450
-Wire Wire Line
-	10350 3950 10750 3950
-Wire Wire Line
-	10050 3700 10250 3700
+	10450 3450 10250 3450
+Wire Wire Line
+	10250 3450 10250 3950
+$Comp
+L Jumper_NO_Small JP_MPU_FSYNC1
+U 1 1 598A250E
+P 10400 3950
+F 0 "JP_MPU_FSYNC1" H 10400 4030 50  0000 C CNN
+F 1 "JP_NO" H 10410 3890 50  0000 C CNN
+F 2 "jumper:SOLDER-JUMPER_1-WAY" H 10400 3950 50  0001 C CNN
+F 3 "" H 10400 3950 50  0000 C CNN
+	1    10400 3950
+	1    0    0    -1
+$EndComp
+Connection ~ 10250 3700
+Wire Wire Line
+	10250 3950 10300 3950
+Wire Wire Line
+	10500 3950 10750 3950
+$Comp
+L C C10
+U 1 1 598A2A36
+P 4100 3850
+F 0 "C10" H 4125 3950 50  0000 L CNN
+F 1 ".1uF" H 4125 3750 50  0000 L CNN
+F 2 "Capacitors_SMD:C_0603_HandSoldering" H 4138 3700 50  0001 C CNN
+F 3 "" H 4100 3850 50  0000 C CNN
+	1    4100 3850
+	-1   0    0    -1
+$EndComp
+Wire Wire Line
+	4000 4500 4750 4500
+Wire Wire Line
+	4100 3200 4100 3700
+Connection ~ 4100 3200
+Connection ~ 4100 4500
+Wire Wire Line
+	4000 3200 4750 3200
+Wire Wire Line
+	4100 4000 4100 4500
+$Comp
+L MAX98357A I2S
+U 1 1 598A3B3F
+P 5150 6700
+F 0 "I2S" H 5150 6600 50  0000 C CNN
+F 1 "MAX98357A" H 5150 6800 50  0000 C CNN
+F 2 "MODULE" H 5150 6700 50  0001 C CNN
+F 3 "DOCUMENTATION" H 5150 6700 50  0001 C CNN
+	1    5150 6700
+	1    0    0    -1
+$EndComp
+$Comp
+L CONN_01X02 SPK
+U 1 1 598A3DF5
+P 6550 6850
+F 0 "SPK" H 6550 7000 50  0000 C CNN
+F 1 "CONN_SPK" V 6650 6850 50  0000 C CNN
+F 2 "" H 6550 6850 50  0000 C CNN
+F 3 "" H 6550 6850 50  0000 C CNN
+	1    6550 6850
+	1    0    0    -1
+$EndComp
+Text GLabel 5150 6000 1    60   Input ~ 0
+5V
+Wire Wire Line
+	5150 6000 5250 6000
+Text GLabel 5050 7400 3    60   Input ~ 0
+GND
+Wire Wire Line
+	5050 7400 5250 7400
+Connection ~ 5150 7400
+$Comp
+L R R4
+U 1 1 598A454E
+P 3800 6600
+F 0 "R4" V 3880 6600 50  0000 C CNN
+F 1 "100K" V 3800 6600 50  0000 C CNN
+F 2 "Resistors_SMD:R_0603_HandSoldering" V 3730 6600 50  0001 C CNN
+F 3 "" H 3800 6600 50  0000 C CNN
+	1    3800 6600
+	0    1    1    0
+$EndComp
+Text GLabel 3650 6600 0    60   Input ~ 0
+GND
+Text GLabel 3650 6700 0    60   Input ~ 0
+5V
+Wire Wire Line
+	3650 6700 3950 6700
+Wire Wire Line
+	3650 6800 3950 6800
+Wire Wire Line
+	3650 6900 3950 6900
+Text GLabel 3650 6500 0    60   Input ~ 0
+ADC_0
+Wire Wire Line
+	3650 6500 3950 6500
+Text GLabel 3650 6800 0    60   Input ~ 0
+ADC_1
+Text GLabel 3650 6900 0    60   Input ~ 0
+ADC_2
 $EndSCHEMATC

Commit message: Finished board layout
Parts:
- removed C9: .1uF, Capacitors_SMD:C_0603_HandSoldering, symbol C
- removed LED1, LED2: WS2812B_LED, LEDs:LED_WS2812B-PLCC4, symbol WS2812B_LED
- removed R2: 100K, Resistors_SMD:R_0603_HandSoldering, symbol R
- added C12, C13: .1uF, Capacitors_SMD:C_0603_HandSoldering, symbol C
- added C9: CP2102, Housings_DFN_QFN:QFN-28-1EP_5x5mm_Pitch0.5mm, symbol CP2102
- added P3: USB_OTG, Connectors_USB:USB_Micro-B_Molex_47346-0001, symbol USB_OTG
- added R5, R6, R7, R8: 1K, Resistors_SMD:R_0603_HandSoldering, symbol R
- I2S1: renamed from I2S; footprint MODULE -> Housings_DFN_QFN:QFN-16-1EP_3x3mm_Pitch0.5mm
- PROG1: renamed from FTDI1; value CONN_FTDI -> PROG
- SERIAL1: renamed from U1; value SERIAL2 -> SERIAL
- SPK1: renamed from SPK; footprint (none) -> Pin_Headers:Pin_Header_Straight_1x02
- renumbered JP_MPU_FSYNC1 to FSYNC1, JP_MPU_INT1 to INT1, WS2812 to WS1
Connections:
- net TOUCH_7 is gone; now on net PROG_DTR: ESP1.25 (IO0), P2.10 (P10)
- net WS2812_OUT is gone; now on net PROG_DTR: WS1.3 (P3)
- net +3V3: now also C13.2, C9.6 (Vdd), C9.7 (REGIN)
- net +5V: now also C12.1
- net ADC_0: no longer I2S1.1 (DIN)
- net ADC_1: no longer I2S1.14 (LRCLK)
- net ADC_2: no longer I2S1.16 (BCLK)
- net ADC_3: now also I2S1.14 (LRCLK)
- net ADC_4: now also I2S1.16 (BCLK)
- net ADC_5: now also I2S1.1 (DIN)
- net GND: now also I2S1.17 (GND_PAD), C12.2, C13.1, C9.29 (GND_PAD), C9.3 (GND), P3.5 (GND)
- net SDA: now also ESP1.37 (IO23); no longer ESP1.33 (IO21)
- net SPI_MOSI: now also ESP1.33 (IO21); no longer ESP1.37 (IO23)
- net FTDI_DTR renamed PROG_DTR
- net PROG_DTR: now also R5.2
- net FTDI_RTS renamed PROG_RTS
- net PROG_RTS: now also R8.2
- net U0_RX renamed PROG_RX
- net PROG_RX: now also ESP1.35 (TXD0), R7.2; no longer ESP1.34 (RXD0)
- net U0_TX renamed PROG_TX
- net PROG_TX: now also ESP1.34 (RXD0), R6.2; no longer ESP1.35 (TXD0)
- new net: C9.8 (VBUS), P3.1 (VBUS)
- new net: C9.5 (D-), P3.2 (D-)
- new net: C9.4 (D+), P3.3 (D+)
- new net: C9.28 (DTR), R5.1
- new net: C9.26 (TXD), R6.1
- new net: C9.25 (RXD), R7.1
- new net: C9.24 (RTS), R8.1
Other:
- moved on the sheet: BME1, C6
